File: buttons-board/buttons-board.kicad_pcb (KiCad board)
At the start: 2 copper layers, 149 x 8 mm, 5 parts, among them J1 Conn_01x05, SW1 SW_Push, SW2 SW_Push, SW3 SW_Push, SW4 SW_Push

Commit message: ground plane
Connections:
- net Net-(J1-Pin_1) renamed GND
Routing:
- net GND: track 130.2 -> 1.21 mm
- added copper zone on B.Cu, net GND
Changed lines of the file:
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@@
 			(plot_on_all_layers_selection 0x00000000_00000000_00000000_00000000)
 			(disableapertmacros no)
-			(usegerberextensions no)
+			(usegerberextensions yes)
 			(usegerberattributes yes)
 			(usegerberadvancedattributes yes)
@@
 			(outputformat 1)
 			(mirror no)
-			(drillshape 1)
+			(drillshape 0)
 			(scaleselection 1)
-			(outputdirectory "")
+			(outputdirectory "out")
 		)
 	)
@@
 	(net 1 "Net-(J1-Pin_4)")
 	(net 2 "Net-(J1-Pin_2)")
-	(net 3 "Net-(J1-Pin_1)")
+	(net 3 "GND")
 	(net 4 "Net-(J1-Pin_3)")
 	(net 5 "Net-(J1-Pin_5)")
@@
 			(layers "*.Cu" "*.Mask")
 			(remove_unused_layers no)
-			(net 3 "Net-(J1-Pin_1)")
+			(net 3 "GND")
 			(pinfunction "1")
 			(pintype "passive")
@@
 			(layers "*.Cu" "*.Mask")
 			(remove_unused_layers no)
-			(net 3 "Net-(J1-Pin_1)")
+			(net 3 "GND")
 			(pinfunction "1")
 			(pintype "passive")
@@
 			(layers "*.Cu" "*.Mask")
 			(remove_unused_layers no)
-			(net 3 "Net-(J1-Pin_1)")
+			(net 3 "GND")
 			(pinfunction "1")
 			(pintype "passive")
@@
 			(layers "*.Cu" "*.Mask")
 			(remove_unused_layers no)
-			(net 3 "Net-(J1-Pin_1)")
+			(net 3 "GND")
 			(pinfunction "1")
 			(pintype "passive")
@@
 			(layers "*.Cu" "*.Mask")
 			(remove_unused_layers no)
-			(net 3 "Net-(J1-Pin_1)")
+			(net 3 "GND")
 			(pinfunction "1")
 			(pintype "passive")
@@
 			(layers "*.Cu" "*.Mask")
 			(remove_unused_layers no)
-			(net 3 "Net-(J1-Pin_1)")
+			(net 3 "GND")
 			(pinfunction "1")
 			(pintype "passive")
@@
 			(layers "*.Cu" "*.Mask")
 			(remove_unused_layers no)
-			(net 3 "Net-(J1-Pin_1)")
+			(net 3 "GND")
 			(pinfunction "1")
 			(pintype "passive")
@@
 			(layers "*.Cu" "*.Mask")
 			(remove_unused_layers no)
-			(net 3 "Net-(J1-Pin_1)")
+			(net 3 "GND")
 			(pinfunction "1")
 			(pintype "passive")
@@
 			(layers "*.Cu" "*.Mask")
 			(remove_unused_layers no)
-			(net 3 "Net-(J1-Pin_1)")
+			(net 3 "GND")
 			(pinfunction "Pin_1")
 			(pintype "passive")
@@
 	)
 	(segment
+		(start 133.5 100.5)
+		(end 135.5 102.5)
+		(width 0.3)
+		(layer "F.Cu")
+		(net 1)
+	)
+	(segment
 		(start 167.42 100)
 		(end 167.54 100)
@@
 	)
 	(segment
-		(start 133.5 100.5)
-		(end 135.5 102.5)
+		(start 117 100.5)
+		(end 133.5 100.5)
+		(width 0.3)
+		(layer "F.Cu")
+		(net 1)
+	)
+	(segment
+		(start 108.75 102.25)
+		(end 115.25 102.25)
+		(width 0.3)
+		(layer "F.Cu")
+		(net 1)
+	)
+	(segment
+		(start 166.5 102.5)
+		(end 167.42 101.58)
+		(width 0.3)
+		(layer "F.Cu")
+		(net 1)
+	)
+	(segment
+		(start 135.5 102.5)
+		(end 166.5 102.5)
+		(width 0.3)
+		(layer "F.Cu")
+		(net 1)
+	)
+	(segment
+		(start 115.25 102.25)
+		(end 117 100.5)
 		(width 0.3)
 		(layer "F.Cu")
@@
 	)
 	(segment
-		(start 135.5 102.5)
-		(end 166.5 102.5)
-		(width 0.3)
-		(layer "F.Cu")
-		(net 1)
-	)
-	(segment
-		(start 108.75 102.25)
-		(end 115.25 102.25)
-		(width 0.2)
-		(layer "F.Cu")
-		(net 1)
-	)
-	(segment
-		(start 117 100.5)
-		(end 133.5 100.5)
-		(width 0.3)
-		(layer "F.Cu")
-		(net 1)
-	)
-	(segment
-		(start 115.25 102.25)
-		(end 117 100.5)
-		(width 0.3)
-		(layer "F.Cu")
-		(net 1)
-	)
-	(segment
-		(start 166.5 102.5)
-		(end 167.42 101.58)
-		(width 0.3)
-		(layer "F.Cu")
-		(net 1)
-	)
-	(segment
 		(start 172.5 100)
 		(end 172.62 100)
@@
 		(start 213.35 102.25)
 		(end 206.85 102.25)
-		(width 0.2)
+		(width 0.3)
 		(layer "F.Cu")
 		(net 2)
-	)
-	(segment
-		(start 175.16 98.66)
-		(end 175.16 100)
-		(width 0.3)
-		(layer "F.Cu")
-		(net 3)
-	)
-	(segment
-		(start 130.25 97.75)
-		(end 131 97)
-		(width 0.3)
-		(layer "F.Cu")
-		(net 3)
-	)
-	(segment
-		(start 108.75 97.75)
-		(end 115.25 97.75)
-		(width 0.3)
-		(layer "F.Cu")
-		(net 3)
-	)
-	(segment
-		(start 206.75 97.75)
-		(end 206.5 97.5)
-		(width 0.3)
-		(layer "F.Cu")
-		(net 3)
 	)
 	(segment
@@
 	)
 	(segment
-		(start 93.5 97.5)
-		(end 108.5 97.5)
-		(width 0.3)
-		(layer "F.Cu")
-		(net 3)
-	)
-	(segment
 		(start 93.25 97.75)
 		(end 93.75 97.75)
@@
 	)
 	(segment
-		(start 86.75 97.75)
-		(end 93.25 97.75)
-		(width 0.3)
-		(layer "F.Cu")
-		(net 3)
-	)
-	(segment
-		(start 213.35 97.75)
-		(end 206.85 97.75)
-		(width 0.2)
-		(layer "F.Cu")
-		(net 3)
-	)
-	(segment
-		(start 115.25 97.75)
-		(end 123.75 97.75)
-		(width 0.3)
-		(layer "F.Cu")
-		(net 3)
-	)
-	(segment
-		(start 131 97)
-		(end 173.5 97)
-		(width 0.3)
-		(layer "F.Cu")
-		(net 3)
-	)
-	(segment
-		(start 206.85 97.75)
-		(end 206.75 97.75)
-		(width 0.3)
-		(layer "F.Cu")
-		(net 3)
-	)
-	(segment
-		(start 176.32 97.5)
-		(end 175.16 98.66)
-		(width 0.3)
-		(layer "F.Cu")
-		(net 3)
-	)
-	(segment
-		(start 206.5 97.5)
-		(end 176.32 97.5)
-		(width 0.3)
-		(layer "F.Cu")
-		(net 3)
-	)
-	(segment
-		(start 123.75 97.75)
-		(end 130.25 97.75)
-		(width 0.3)
-		(layer "F.Cu")
-		(net 3)
-	)
-	(segment
-		(start 173.5 97)
-		(end 175.16 98.66)
-		(width 0.3)
-		(layer "F.Cu")
-		(net 3)
-	)
-	(segment
 		(start 168.5 103)
 		(end 169.96 101.54)
@@
 		(start 123.75 102.25)
 		(end 130.25 102.25)
-		(width 0.2)
+		(width 0.3)
 		(layer "F.Cu")
 		(net 4)
@@
 	)
 	(segment
-		(start 105.5 102.5)
-		(end 108.5 99.5)
+		(start 133 100)
+		(end 135.301 97.699)
 		(width 0.3)
 		(layer "F.Cu")
@@
 	)
 	(segment
-		(start 164 97.5)
-		(end 164.88 98.38)
+		(start 163.699 97.699)
+		(end 164.88 98.88)
 		(width 0.3)
 		(layer "F.Cu")
@@
 	)
 	(segment
+		(start 164.88 98.88)
+		(end 164.88 100)
+		(width 0.3)
+		(layer "F.Cu")
+		(net 5)
+	)
+	(segment
 		(start 93.25 102.25)
-		(end 93.5 102.5)
-		(width 0.3)
-		(layer "F.Cu")
-		(net 5)
-	)
-	(segment
-		(start 135.5 97.5)
-		(end 164 97.5)
-		(width 0.3)
-		(layer "F.Cu")
-		(net 5)
-	)
-	(segment
-		(start 93.5 102.5)
-		(end 105.5 102.5)
-		(width 0.3)
-		(layer "F.Cu")
-		(net 5)
-	)
-	(segment
-		(start 108.5 99.5)
-		(end 133.5 99.5)
-		(width 0.3)
-		(layer "F.Cu")
-		(net 5)
-	)
-	(segment
-		(start 133.5 99.5)
-		(end 135.5 97.5)
+		(end 96.25 102.25)
 		(width 0.3)
 		(layer "F.Cu")
@@
 	)
 	(segment
-		(start 164.88 98.38)
-		(end 164.88 100)
+		(start 108 100)
+		(end 133 100)
+		(width 0.3)
+		(layer "F.Cu")
+		(net 5)
+	)
+	(segment
+		(start 97 103)
+		(end 105 103)
 		(width 0.3)
 		(layer "F.Cu")
@@
 		(net 5)
 	)
+	(segment
+		(start 96.25 102.25)
+		(end 97 103)
+		(width 0.3)
+		(layer "F.Cu")
+		(net 5)
+	)
+	(segment
+		(start 135.301 97.699)
+		(end 163.699 97.699)
+		(width 0.3)
+		(layer "F.Cu")
+		(net 5)
+	)
+	(segment
+		(start 105 103)
+		(end 108 100)
+		(width 0.3)
+		(layer "F.Cu")
+		(net 5)
+	)
+	(zone
+		(net 3)
+		(net_name "GND")
+		(layer "B.Cu")
+		(hatch edge 0.5)
+		(connect_pads
+			(clearance 0.5)
+		)
+		(min_thickness 0.25)
+		(filled_areas_thickness no)
+		(fill yes
+			(thermal_gap 0.5)
+			(thermal_bridge_width 0.5)
+		)
+		(polygon
+			(pts
+				(xy 74 94) (xy 226 94) (xy 226 106) (xy 74 106)
+			)
+		)
+	)
 	(embedded_fonts no)

Commit message: pcb
Parts:
- removed the SW1 at (86.8, 97.8)
- J1: footprint Connector_PinHeader_2.54mm:PinHeader_1x05_P2.54mm_Vertical -> Connector_PinHeader_2.54mm:PinHeader_1x04_P2.54mm_Horizontal
- moved SW1 19.6 mm to (89.1, 97.8)
- moved SW2 19.4 mm to (104.4, 97.8)
- moved J1 12.7 mm to (162.3, 100.0)
- moved SW3 2.48 mm to (204.4, 97.8)
- renumbered SW2 to SW1, SW3 to SW2, SW4 to SW3
Routing:
- net Net-(J1-Pin_5): track 82.4 -> 0.00 mm
- net Net-(J1-Pin_2): track 43.0 -> 53.8 mm
- net Net-(J1-Pin_3): track 48.8 -> 55.5 mm
- net Net-(J1-Pin_4): track 62.3 -> 68.6 mm
- net GND: track 1.21 -> 0.00 mm
Other:
- outline, holes or cut-outs redrawn
- board text added: "${REFERENCE}"

Commit message: pcb final
Other:
- board text removed: "${REFERENCE}"
Changed lines of the file:
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@@
 	(title_block
 		(title "Buttons board")
+		(date "2026-02-21")
+		(rev "1.0")
 		(company "StrangePlanet")
 	)
@@
 		)
 	)
-	(gr_circle
-		(center 162.3 101.8)
-		(end 162.7 101.8)
+	(gr_poly
+		(pts
+			(xy 161.798 102.362) (xy 162.814 102.362) (xy 162.306 101.854)
+		)
 		(stroke
 			(width 0.1)
@@
 		(layer "Edge.Cuts")
 	)
-	(gr_text "${REFERENCE}"
-		(at 171.23 97.23 0)
-		(layer "B.Fab")
-		(effects
-			(font
-				(size 1 1)
-				(thickness 0.15)
-			)
-			(justify mirror)
-		)
-	)
 	(segment
