File: buttons-board/buttons-board.kicad_sch (KiCad schematic)
At the start: 5 parts, among them J1 Conn_01x05, SW1 SW_Push, SW2 SW_Push, SW3 SW_Push, SW4 SW_Push

Commit message: ground plane
Connections:
- net GND: now reaches J1.1 (Pin_1), SW1.1, SW2.1, SW3.1, SW4.1
Changed lines of the file:
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@@
+	)
+	(junction
+		(at 138.43 116.84)
+		(diameter 0)
+		(color 0 0 0 0)
 	)
 	(junction
@@
 	(wire
 		(pts
+			(xy 138.43 116.84) (xy 128.27 116.84)
+		)
+		(stroke
+			(width 0)
+			(type default)
+		)
+	)
+	(wire
+		(pts
 			(xy 128.27 92.71) (xy 128.27 102.87)
 		)
@@
 	(wire
 		(pts
-			(xy 147.32 116.84) (xy 128.27 116.84)
+			(xy 147.32 116.84) (xy 138.43 116.84)
 		)
 		(stroke
@@
 					(unit 1)
 				)
+			)
+		)
+	)
+	(symbol
+		(lib_id "power:GND")
+		(at 138.43 116.84 0)
+		(unit 1)
+		(exclude_from_sim no)
+		(in_bom yes)
+		(on_board yes)
+		(dnp no)
+		(fields_autoplaced yes)
+		(property "Reference" "#PWR01"
+			(at 138.43 123.19 0)
+			(effects
+				(font
+					(size 1.27 1.27)
+				)
+				(hide yes)
+			)
+		)
+		(property "Value" "GND"
+			(at 138.43 121.92 0)
+			(effects
+				(font
+					(size 1.27 1.27)
+				)
+			)
+		)
+		(property "Footprint" ""
+			(at 138.43 116.84 0)
+			(effects
+				(font
+					(size 1.27 1.27)
+				)
+				(hide yes)
+			)
+		)
+		(property "Datasheet" ""
+			(at 138.43 116.84 0)
+			(effects
+				(font
+					(size 1.27 1.27)
+				)
+				(hide yes)
+			)
+		)
+		(property "Description" "Power symbol creates a global label with name \"GND\" , ground"
+			(at 138.43 116.84 0)
+			(effects
+				(font
+					(size 1.27 1.27)
+				)
+				(hide yes)
+			)
+		)
+		(pin "1"
+		)
+		(instances
+			(project ""
+				(path "/bb57ecba-c46e-4ba4-90ac-09edad2d3bfa"
+					(reference "#PWR01")
+					(unit 1)
+				)

Commit message: pcb
Parts:
- removed SW1: SW_Push, Button_Switch_THT:SW_PUSH_6mm_H4.3mm, symbol Switch:SW_Push
- J1: footprint Connector_PinHeader_2.54mm:PinHeader_1x05_P2.54mm_Vertical -> Connector_PinHeader_2.54mm:PinHeader_1x04_P2.54mm_Horizontal; symbol Connector_Generic:Conn_01x05 -> Connector_Generic:Conn_01x04
- renumbered SW2 to SW1, SW3 to SW2, SW4 to SW3
Other:
- moved on the sheet: SW1, SW2, SW3

Commit message: pcb final
Other:
- moved on the sheet: J1, SW1, SW2, SW3
