File: main-board/in-2-nixie.kicad_pcb (KiCad board)
At the start: 2 copper layers, 167 x 52 mm, 26 parts, among them J1 Encoder, J2 Matrix, J3 Power, J4 DS3231, J5 Buttons, T1 IN-2, T2 IN-2, T3 IN-2, T4 IN-2, U1 HV5222PJ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

Commit message: pcb
Parts:
- removed C2: 10n, Capacitor_THT:C_Disc_D5.0mm_W2.5mm_P5.00mm
- removed the J4 at (96.2, 79.0)
- removed R7: 10k, Resistor_THT:R_Axial_DIN0207_L6.3mm_D2.5mm_P7.62mm_Horizontal
- added D1: 1N4148, Diode_THT:D_DO-35_SOD27_P7.62mm_Horizontal, F.Cu at (97.3, 51.3)
- added D2: WS2812B, in-2-nixie:APA106_D5-Staggered_Pins, F.Cu at (142.4, 56.6)
- added D3: WS2812B, in-2-nixie:APA106_D5-Staggered_Pins, F.Cu at (162.4, 56.6)
- added D4: WS2812B, in-2-nixie:APA106_D5-Staggered_Pins, F.Cu at (192.4, 56.6)
- added D5: WS2812B, in-2-nixie:APA106_D5-Staggered_Pins, F.Cu at (212.4, 56.6)
- added J5: BME280, Connector_PinHeader_2.54mm:PinHeader_1x04_P2.54mm_Vertical, B.Cu at (103.6, 82.8)
- added J6: DS3231, Connector_PinHeader_2.54mm:PinHeader_1x05_P2.54mm_Vertical, B.Cu at (93.0, 98.0)
- added Q1: MPSA42, Package_TO_SOT_THT:TO-92_Inline, F.Cu at (160.3, 92.2)
- added R10: 33k, Resistor_THT:R_Axial_DIN0207_L6.3mm_D2.5mm_P2.54mm_Vertical, F.Cu at (153.9, 90.9)
- added R6: 10k, Resistor_THT:R_Axial_DIN0207_L6.3mm_D2.5mm_P2.54mm_Vertical, F.Cu at (190.2, 97.0)
- C1: value 10n -> 330u; footprint Capacitor_THT:C_Disc_D5.0mm_W2.5mm_P5.00mm -> Capacitor_THT:CP_Radial_D8.0mm_P3.50mm
- J1: footprint Connector_PinHeader_2.54mm:PinHeader_1x03_P2.54mm_Vertical -> Connector_PinHeader_2.54mm:PinHeader_1x04_P2.54mm_Vertical
- J3: renamed from J5; footprint Connector_PinHeader_2.54mm:PinHeader_1x05_P2.54mm_Vertical -> Connector_PinHeader_2.54mm:PinHeader_1x04_P2.54mm_Vertical
- R1, R2, R4, R5: value R -> 10k
- R3: value R -> 200k
- R8: value 20k -> 10k; footprint Resistor_THT:R_Axial_DIN0207_L6.3mm_D2.5mm_P7.62mm_Horizontal -> Resistor_THT:R_Axial_DIN0207_L6.3mm_D2.5mm_P2.54mm_Vertical
- R9: value 20k -> 200k
- U3: value ESP32-C6 -> ESP32-C6 SuperMini
- moved R9 106.2 mm to (182.6, 68.1)
- moved R8 86.6 mm to (164.1, 97.0), turned to 0 degrees
- moved C1 49.8 mm to (131.8, 83.0), turned to 135 degrees
- moved J2 19.7 mm to (103.6, 79.5), turned to -90 degrees
- moved J1 10.5 mm to (86.6, 78.0), turned to 0 degrees
- moved C3 7.63 mm to (194.6, 97.0)
- moved R5 7.22 mm to (208.5, 62.5), turned to 15 degrees
- moved R2 7.19 mm to (158.5, 62.5), turned to 15 degrees
- moved R4 7.17 mm to (188.5, 62.5), turned to 15 degrees
- moved R1 7.14 mm to (138.4, 62.5), turned to 15 degrees
- moved U4 6.87 mm to (114.0, 91.0)
- moved J3 4.63 mm to (116.1, 74.4), turned to 180 degrees
- moved J4 2.91 mm to (122.2, 59.2), turned to 0 degrees
- moved R3 1.57 mm to (172.0, 68.1)
- moved L1 0.50 mm to (177.4, 66.6), turned to 90 degrees
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- renumbered J3 to J4
Connections:
- C1 pad 1: /ROT_B -> +5V
- J1 pad 2: Net-(J1-Pin_2) -> /ROT_SW
- J1 pad 3: Net-(J1-Pin_3) -> /ROT_B
- J3 pad 2: /BTN_4 -> /BTN_3
- J3 pad 3: /BTN_3 -> /BTN_2
- J3 pad 4: /BTN_2 -> /BTN_1
- L2 pad 1: Net-(L2-K) -> Net-(L1-K)
- L2 pad 2: Net-(L1-K) -> Net-(L2-A)
- R8 pad 1: /ROT_A -> GND
- R8 pad 2: Net-(J1-Pin_3) -> /NIXIE_EN
- R9 pad 1: /ROT_B -> Net-(L2-A)
- R9 pad 2: Net-(J1-Pin_2) -> Net-(U2-HV)
- U1 pad 2: Net-(L2-K) -> unconnected-(U1B-HVOUT16-Pad2)
- U1 pad 27: +5V -> Net-(U1A-STR)
- U2 pad 2: Net-(U2-EN) -> unconnected-(U2-EN-Pad2)
- U3 pad 14: /BTN_4 -> /ROT_B
- U3 pad 20: /BTN_2 -> /ROT_A
- U3 pad 22: /ROT_B -> /BTN_2
- U3 pad 26: +5V -> Net-(D1-K)
- U3 pad 3: /BTN_1 -> Net-(U3-GPIO3)
- U3 pad 4: unconnected-(U3-GPIO4-Pad4) -> /BTN_1
- U3 pad 5: unconnected-(U3-GPIO5-Pad5) -> /BTN_3
- U3 pad 8: unconnected-(U3-GPIO8-Pad8) -> /LEDS
- U3 pad 9: unconnected-(U3-GPIO9-Pad9) -> /ROT_SW
- U4 pad 10: /NIXIE_CLK -> /NIXIE_DIN
- U4 pad 11: /NIXIE_DIN -> /NIXIE_DOT
- U4 pad 2: Net-(U3-GPIO0) -> Net-(U3-GPIO3)
- U4 pad 3: Net-(U3-GPIO1) -> Net-(U3-GPIO2)
- U4 pad 4: Net-(U3-GPIO2) -> Net-(U3-GPIO1)
- U4 pad 5: unconnected-(U4-A4-Pad5) -> Net-(U3-GPIO0)
- U4 pad 8: unconnected-(U4-B4-Pad8) -> /NIXIE_EN
- U4 pad 9: /NIXIE_EN -> /NIXIE_CLK
Routing:
- net +5V: track 159.2 -> 270.3 mm
- net /LEDS: track 0.00 -> 59.3 mm, vias 0 -> 2
- net /NIXIE_DOT: track 0.00 -> 38.6 mm
- net /BTN_4: track 32.6 -> 0.00 mm
- net /ROT_B: track 35.8 -> 8.36 mm, vias 1 -> 0
- net Net-(L1-K): track 10.0 -> 36.3 mm
- net Net-(D3-DOUT): track 0.00 -> 25.8 mm
- net Net-(U3-GPIO3): track 0.00 -> 24.8 mm
- net /ROT_A: track 39.1 -> 15.9 mm, vias 1 -> 0
- net /BTN_2: track 38.7 -> 19.5 mm
- net Net-(D4-DOUT): track 0.00 -> 15.8 mm
- net Net-(D2-DOUT): track 0.00 -> 15.8 mm
- net /BTN_1: track 23.0 -> 7.39 mm
- net /BTN_3: track 19.3 -> 8.42 mm
- net Net-(U1A-STR): track 0.00 -> 9.74 mm, vias 0 -> 1
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Other:
- outline, holes or cut-outs redrawn
- board text added: "BME280"
- board text added: "Buttons"
- board text added: "DS3231"
- board text added: "Encoder"
- board text added: "Matrix"
- board text added: "© StrangePlanet 2026"

Commit message: update
Parts:
- moved J6 10.6 mm to (103.6, 98.0)
- moved U4 2.10 mm to (114.0, 88.9)
- moved Q1 1.61 mm to (158.8, 91.7)
- moved C1 1.45 mm to (131.8, 84.5), turned to 180 degrees
- moved R10 0.74 mm to (154.4, 91.4), turned to 90 degrees
- moved R8 0.25 mm to (163.8, 97.0)
Connections:
- R8 pad 1: GND -> /NIXIE_EN
- R8 pad 2: /NIXIE_EN -> GND
- T1 pad 3: unconnected-(T1-K3-Pad3) -> Net-(T1-K3)
- T1 pad 4: unconnected-(T1-K4-Pad4) -> Net-(T1-K4)
- T1 pad 5: unconnected-(T1-K5-Pad5) -> Net-(T1-K5)
- U1 pad 10: Net-(T2-K8) -> Net-(T2-K9)
- U1 pad 11: Net-(T2-K9) -> Net-(T2-K0)
- U1 pad 12: Net-(T2-K0) -> Net-(T1-K5)
- U1 pad 13: Net-(T1-K2) -> Net-(T1-K4)
- U1 pad 14: Net-(T1-K1) -> Net-(T1-K3)
- U1 pad 15: Net-(T1-K0) -> Net-(T1-K2)
- U1 pad 16: unconnected-(U1B-HVOUT2-Pad16) -> Net-(T1-K1)
- U1 pad 17: unconnected-(U1B-HVOUT1-Pad17) -> Net-(T1-K0)
- U1 pad 2: unconnected-(U1B-HVOUT16-Pad2) -> Net-(T2-K6)
- U1 pad 3: Net-(T2-K6) -> Net-(T2-K5)
- U1 pad 4: Net-(T2-K5) -> Net-(T2-K4)
- U1 pad 5: Net-(T2-K4) -> Net-(T2-K3)
- U1 pad 6: Net-(T2-K3) -> Net-(T2-K2)
- U1 pad 7: Net-(T2-K2) -> Net-(T2-K1)
- U1 pad 8: Net-(T2-K1) -> Net-(T2-K7)
- U1 pad 9: Net-(T2-K7) -> Net-(T2-K8)
Routing:
- net Net-(T1-K5): track 0.00 -> 30.9 mm
- net Net-(T1-K3): track 0.00 -> 30.0 mm
- net Net-(T1-K4): track 0.00 -> 29.8 mm
- net +5V: track 270.3 -> 258.7 mm
- net /LEDS: track 59.3 -> 63.1 mm, vias 2 -> 1
- net /SDA: track 28.6 -> 31.5 mm
- net Net-(U3-GPIO0): track 41.3 -> 38.7 mm
- net Net-(U3-GPIO2): track 30.3 -> 27.7 mm
- net Net-(U3-GPIO3): track 24.8 -> 22.2 mm
- net Net-(U3-GPIO1): track 35.8 -> 33.2 mm
- net Net-(T4-K7): track 38.6 -> 40.4 mm
- net Net-(T2-K3): track 11.8 -> 10.1 mm
- net Net-(T2-K4): track 14.0 -> 12.3 mm
- net Net-(T4-K6): track 40.2 -> 41.9 mm
- net Net-(T4-K5): track 40.5 -> 42.0 mm
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Other:
- outline, holes or cut-outs redrawn

Commit message: pcb final
Parts:
- added G***: LOGO, in-2-nixie:sp_logo, B.Cu at (202.1, 86.3)
Connections:
- J2 pad 1: +5V -> +3.3V
- J5 pad 1: +5V -> +3.3V
- J6 pad 5: +5V -> +3.3V
Routing:
- net +5V: track 258.7 -> 234.2 mm
- net +3.3V: track 37.1 -> 46.1 mm
- net GND: track 1.81 -> 1.78 mm, vias 54 -> 60
Other:
- board text added: "${TITLE} ${REVISION} © ${COMPANY} 2026"
- board text removed: "© StrangePlanet 2026"

Commit message: fix encoder routing
Connections:
- J1 pad 2: /ROT_SW -> /ROT_A
- J1 pad 4: /ROT_A -> /ROT_SW
- U3 pad 20: /ROT_A -> /ROT_SW
- U3 pad 9: /ROT_SW -> /ROT_A
Routing:
- net /ROT_SW: track 8.36 -> 15.9 mm
- net /ROT_A: track 15.9 -> 8.36 mm
Changed lines of the file:
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@@
 			(layers "*.Cu" "*.Mask")
 			(remove_unused_layers no)
-			(net 80 "/ROT_SW")
+			(net 3 "/ROT_A")
 			(pinfunction "GPIO9")
 			(pintype "bidirectional")
@@
 			(layers "*.Cu" "*.Mask")
 			(remove_unused_layers no)
-			(net 3 "/ROT_A")
+			(net 80 "/ROT_SW")
 			(pinfunction "GPIO20")
 			(pintype "bidirectional")
@@
 			(layers "*.Cu" "*.Mask")
 			(remove_unused_layers no)
-			(net 80 "/ROT_SW")
+			(net 3 "/ROT_A")
 			(pinfunction "Pin_2")
 			(pintype "passive")
@@
 			(layers "*.Cu" "*.Mask")
 			(remove_unused_layers no)
-			(net 3 "/ROT_A")
+			(net 80 "/ROT_SW")
 			(pinfunction "Pin_4")
 			(pintype "passive")
@@
 	)
 	(segment
-		(start 91.694 60.846)
-		(end 93.46 59.08)
-		(width 0.2)
-		(layer "F.Cu")
-		(net 3)
-	)
-	(segment
-		(start 86.614 70.358)
-		(end 89.662 70.358)
-		(width 0.2)
-		(layer "F.Cu")
-		(net 3)
-	)
-	(segment
-		(start 89.662 70.358)
-		(end 91.694 68.326)
+		(start 90.272 71.78)
+		(end 93.46 71.78)
 		(width 0.2)
 		(layer "F.Cu")
@@
 	)
 	(segment
-		(start 91.694 68.326)
-		(end 91.694 60.846)
+		(start 86.614 75.438)
+		(end 90.272 71.78)
 		(width 0.2)
 		(layer "F.Cu")
@@
 	)
 	(segment
-		(start 90.272 71.78)
-		(end 93.46 71.78)
+		(start 91.694 60.846)
+		(end 93.46 59.08)
 		(width 0.2)
 		(layer "F.Cu")
@@
 	)
 	(segment
-		(start 86.614 75.438)
-		(end 90.272 71.78)
+		(start 86.614 70.358)
+		(end 89.662 70.358)
+		(width 0.2)
+		(layer "F.Cu")
+		(net 80)
+	)
+	(segment
+		(start 89.662 70.358)
+		(end 91.694 68.326)
+		(width 0.2)
+		(layer "F.Cu")
+		(net 80)
+	)
+	(segment
+		(start 91.694 68.326)
+		(end 91.694 60.846)
 		(width 0.2)
 		(layer "F.Cu")
